File: QSE-Filter.kicad_sch (KiCad schematic)
At the start: 63 parts, among them J1 5-1814832-1, J2 5-1814832-1, J4 Conn_02x05_Odd_Even, U1 MASWSS0179, U10 MASWSS0179, U12 4002, U2 MASWSS0179, U3 MASWSS0179, U4 MASWSS0179, U5 MASWSS0179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

Commit message: Updated schematic with toroid winding information.
Other:
- note added: "10 AND 15 METER COILS USE AWG#27"
- note added: "80 40 AND 20 METER COILS USE AWG#28"
- note added: "T-37-17 8 TURNS"
- note added: "T-37-17 9 TURNS"
- note added: "T-37-6 13 TURNS"
- note added: "T-37-6 18 TURNS"
- note added: "T-37-6 9 TURNS"
- note removed: "T-37-6 XX TURNS"
